File: Keyboard/Keyboard.brd (EAGLE design)
At the start: 324 x 112 mm, 147 parts

Commit message: slight change to keyboard, teensy 3.2
Parts:
- removed J1: (no value), SparkFun-Connectors:1X17
- added B1: TEENSY-3.1SILK, SparkFun-Boards:TEENSY-3.1
- moved D34 59.5 mm to (104.7, 17.8)
- moved D33 51.9 mm to (159.1, 17.8)
- moved J3 35.5 mm to (14.5, 93.7), turned to 0 degrees
- moved D64 20.4 mm to (271.1, 36.8), turned to 180 degrees
- moved D8 11.0 mm to (9.73, 55.9)
- moved D69 10.2 mm to (263.5, 17.8)
- moved D30 8.04 mm to (281.5, 17.8)
- moved D26 7.67 mm to (117.4, 17.8)
- moved D35 5.80 mm to (216.2, 17.8)
- moved D36 5.10 mm to (172.8, 17.8)
- moved D70 5.08 mm to (238.1, 17.8)
- moved D24 5.08 mm to (66.6, 17.8)
- moved D32 3.75 mm to (78.3, 17.8)
- moved D29 3.73 mm to (250.3, 17.8)
- moved D31 2.66 mm to (52.4, 17.8)
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Connections:
- new net 3.3V: B1.3.3V
- new net 3V: B1.3V
- new net AGND: B1.AGND
- new net GND: B1.GND
- new net GND1: B1.GND1
- new net VBAT: B1.VBAT
- new net VIN: B1.VIN
- new net VUSB: B1.VUSB
- net KEYCOLUM0: now also B1.14; no longer J1.7
- net KEYCOLUM1: now also B1.15; no longer J1.6
- net KEYCOLUM2: now also B1.16, B1.17; no longer J1.5
- net KEYCOLUM3: no longer J1.4
- net KEYCOLUM4: now also B1.20; no longer J1.3
- net KEYCOLUM5: now also B1.21; no longer J1.2
- net KEYCOLUM6: now also B1.22, B1.A10; no longer J1.1
- net KEYROW0: now also B1.0; no longer J1.17
- net KEYROW1: now also B1.1; no longer J1.16
- net KEYROW2: now also B1.2; no longer J1.15
- net KEYROW3: now also B1.3; no longer J1.14
- net KEYROW4: now also B1.4; no longer J1.13
- net KEYROW5: now also B1.5; no longer J1.12
- net KEYROW6: now also B1.6; no longer J1.11
- net KEYROW7: now also B1.7; no longer J1.10
- net KEYROW8: now also B1.8; no longer J1.9
- net KEYROW9: now also B1.9; no longer J1.8
Routing:
- net KEYCOLUM1: track 0.00 -> 607.0 mm, vias 0 -> 5
- net KEYCOLUM6: track 0.00 -> 596.4 mm, vias 0 -> 6
- net KEYCOLUM5: track 0.00 -> 592.1 mm, vias 0 -> 6
- net KEYCOLUM4: track 0.00 -> 566.1 mm, vias 0 -> 9
- net KEYROW9: track 0.00 -> 552.9 mm
- net KEYCOLUM2: track 0.00 -> 526.9 mm, vias 0 -> 4
- net KEYCOLUM3: track 0.00 -> 517.7 mm, vias 0 -> 4
- net KEYCOLUM0: track 0.00 -> 510.8 mm, vias 0 -> 6
- net KEYROW7: track 0.00 -> 459.2 mm, vias 0 -> 3
- net KEYROW4: track 0.00 -> 433.8 mm, vias 0 -> 3
- net KEYROW8: track 0.00 -> 362.0 mm, vias 0 -> 5
- net KEYROW6: track 0.00 -> 348.9 mm, vias 0 -> 3
- net KEYROW5: track 0.00 -> 332.2 mm, vias 0 -> 7
- net KEYROW1: track 0.00 -> 293.3 mm, vias 0 -> 2
- net KEYROW3: track 0.00 -> 291.5 mm, vias 0 -> 3
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
Commit message: changed ctrl and alt keyboard position, clean up
Parts:
- moved D21 4.70 mm to (33.5, 55.9)
- moved TAB 4.70 mm to (33.4, 65.4)
- moved D19 2.54 mm to (35.6, 36.8)
- moved CTRL 2.35 mm to (35.7, 46.3)
Routing:
- net KEYROW2: track 283.1 -> 301.6 mm
- net KEYROW3: track 291.5 -> 298.9 mm
- net KEYROW4: track 433.8 -> 441.0 mm
- net N$17: track 10.8 -> 16.7 mm
- net KEYCOLUM3: track 517.7 -> 521.2 mm
- net KEYCOLUM0: track 510.8 -> 514.1 mm
- net N$15: track 10.8 -> 8.92 mm
- net KEYCOLUM2: track 526.9 -> 528.8 mm
